Commit message: urdf gripper

File: src/my_ur_description/urdf/ur_2fg7.urdf.xacro (robot description, xacro)
@@ -1,4 +1,4 @@
 <?xml version="1.0"?>
-<robot xmlns:xacro="http://wiki.ros.org/xacro" name="$(arg name)">
+<robot xmlns:xacro="http://wiki.ros.org/xacro" name="ur">
   <xacro:arg name="name" default="ur"/>
   <xacro:arg name="ur_type" default="ur5e"/>
@@ -39,6 +39,4 @@
   <xacro:include filename="$(find my_ur_description)/urdf/ur_macro.xacro"/>
   <xacro:property name="initial_positions_file" default="$(arg initial_positions_file)"/>
-  <xacro:property name="is_sim_gazebo" value="$(arg sim_gazebo)"/>
-  <xacro:property name="is_sim_ignition" value="$(arg sim_ignition)"/>
   <link name="world" />
   <xacro:ur_robot
@@ -80,4 +78,12 @@
     <origin xyz="0 0 0" rpy="0 0 0" />
   </xacro:ur_robot>
+  <!-- Gazebo ros2_control plugin -->
+  <xacro:if value="$(arg sim_gazebo)">
+    <gazebo>
+      <plugin name="gazebo_ros2_control" filename="libgazebo_ros2_control.so">
+        <parameters>$(arg simulation_controllers)</parameters>
+      </plugin>
+    </gazebo>
+  </xacro:if>
   <!-- Gripper body -->
   <link name="2fg7_base">
@@ -86,5 +92,5 @@
       <geometry>
         <mesh filename="package://my_ur_description/meshes/2fg7.stl"
-              scale="0.001 0.001 0.001"/>
+            scale="0.001 0.001 0.001"/>
       </geometry>
     </visual>
@@ -92,10 +98,22 @@
       <origin xyz="0 0 0" rpy="0 0 0"/>
       <geometry>
-        <mesh filename="package://my_ur_description/meshes/2fg7.stl"
-              scale="0.001 0.001 0.001"/>
+        <box size="0.06 0.06 0.15"/>
       </geometry>
     </collision>
+    <inertial>
+      <origin xyz="0 0 0.075" rpy="0 0 0"/>
+      <mass value="0.8"/>
+      <inertia
+        ixx="0.002"
+        ixy="0.0"
+        ixz="0.0"
+        iyy="0.002"
+        iyz="0.0"
+        izz="0.001"/>
+    </inertial>
   </link>
-  <!-- tool0 to gripper mount -->
+  <gazebo reference="2fg7_base">
+    <material>Gazebo/Red</material>
+  </gazebo>
   <joint name="tool0_to_2fg7_base" type="fixed">
     <parent link="tool0"/>
@@ -103,5 +121,4 @@
     <origin xyz="0 0 0" rpy="0 0 0"/>
   </joint>
-  <!-- TCP of the gripper -->
   <link name="2fg7_tcp"/>
   <joint name="2fg7_base_to_tcp" type="fixed">

Commit message: 2fg7.obj added

File: src/my_ur_description/urdf/ur_2fg7.urdf.xacro (robot description, xacro)
@@ -91,5 +91,5 @@
       <origin xyz="0 0 0" rpy="0 0 0"/>
       <geometry>
-        <mesh filename="package://my_ur_description/meshes/2fg7.stl"
+        <mesh filename="package://my_ur_description/meshes/2fg7.obj"
             scale="0.001 0.001 0.001"/>
       </geometry>

Commit message: gripper a gazebo solved

File: src/my_ur_description/urdf/ur_2fg7.urdf.xacro (robot description, xacro)
@@ -91,6 +91,5 @@
       <origin xyz="0 0 0" rpy="0 0 0"/>
       <geometry>
-        <mesh filename="package://my_ur_description/meshes/2fg7.obj"
-            scale="0.001 0.001 0.001"/>
+        <mesh filename="file://$(find my_ur_description)/meshes/2fg7.stl" scale="0.001 0.001 0.001"/>
       </geometry>
     </visual>
@@ -114,5 +113,5 @@
   </link>
   <gazebo reference="2fg7_base">
-    <material>Gazebo/Red</material>
+    <material>Gazebo/Gray</material>
   </gazebo>
   <joint name="tool0_to_2fg7_base" type="fixed">
